Commit message: Motoman compiling and working

File: resources/motoman/motoman_spherized.urdf (robot description, URDF)
Before this commit: robot motoman_sda10f, 20 links, 19 joints
Links:
- link arm_left_link_1_s: geometry collision sphere radius=0.153255; visual mesh filename=meshes/sda10f/visual/link_s.stl
- link arm_left_link_2_l: geometry collision sphere radius=0.095701; collision sphere radius=0.119311
- link arm_left_link_3_e: geometry collision sphere radius=0.085433; collision sphere radius=0.095372
- link arm_left_link_4_u: geometry collision sphere radius=0.080043; collision sphere radius=0.088818
- link arm_left_link_5_r: geometry collision sphere radius=0.077046; collision sphere radius=0.079093
- link arm_left_link_6_b: geometry collision sphere radius=0.068019; collision sphere radius=0.077881
- link arm_left_link_7_t: geometry collision sphere radius=0.034568; collision sphere radius=0.035041
- link arm_right_link_1_s: geometry collision sphere radius=0.153255; visual mesh filename=meshes/sda10f/visual/link_s.stl
- link arm_right_link_2_l: geometry collision sphere radius=0.095701; collision sphere radius=0.119311
- link arm_right_link_3_e: geometry collision sphere radius=0.085433; collision sphere radius=0.095372
- link arm_right_link_4_u: geometry collision sphere radius=0.080043; collision sphere radius=0.088818
- link arm_right_link_5_r: geometry collision sphere radius=0.077046; collision sphere radius=0.079093
- link arm_right_link_6_b: geometry collision sphere radius=0.068019; collision sphere radius=0.077881
- link arm_right_link_7_t: geometry collision sphere radius=0.034568; collision sphere radius=0.035041
- link torso_base_link: geometry collision sphere radius=0.273417; collision sphere radius=0.325854
- link torso_link_b1: geometry collision sphere radius=0.186756; collision sphere radius=0.187648
