Commit message: refactor

File: resources/panda/bipanda_spherized.urdf (robot description, URDF)
Before this commit: robot bipanda, 27 links, 26 joints
Joints:
- joint left_panda_finger_joint2: mimic joint=left_panda_finger_joint1 -> (none)
- joint right_panda_finger_joint2: mimic joint=right_panda_finger_joint1 -> (none)
