Commit message: updated composer for composite robots, spherical ridgeback approximation

File: resources/ridgeback/ridgeback_spherized.urdf (robot description, URDF)
Before this commit: robot ridgeback, 22 links, 21 joints
Links:
- link mobilebase0_chassis_link: geometry collision sphere radius=0.142467; collision sphere radius=0.166733
- link mobilebase0_riser_link: geometry collision sphere radius=0.049782; collision sphere radius=0.05326
- link mobilebase0_top_link: geometry collision sphere radius=0.078189; collision sphere radius=0.087608

File: resources/ridgebackdualpanda/ridgebackdualpanda.urdf (robot description, URDF)
Before this commit: robot ridgeback_dual_panda, 50 links, 49 joints
Links:
- removed link gripperleft_0_eef
- removed link gripperright_0_eef
- added link gripper0_left_eef
- added link gripper0_right_eef
Joints:
- removed joint gripperleft_0_eef_joint
- removed joint gripperright_0_eef_joint
- added joint gripper0_left_eef_joint: type fixed, parent robot0_left_hand, child gripper0_left_eef, origin xyz=0 0 0.097 rpy=0 0 -1.57079633
- added joint gripper0_right_eef_joint: type fixed, parent robot0_right_hand, child gripper0_right_eef, origin xyz=0 0 0.097 rpy=0 0 -1.57079633

File: resources/ridgebackdualpanda/ridgebackdualpanda_spherized.urdf (robot description, URDF)
Before this commit: robot ridgeback_dual_panda, 50 links, 49 joints
Links:
- removed link gripperleft_0_eef
- removed link gripperright_0_eef
- added link gripper0_left_eef
- added link gripper0_right_eef
- link mobilebase0_chassis_link: geometry collision sphere radius=0.142467; collision sphere radius=0.166733
- link mobilebase0_riser_link: geometry collision sphere radius=0.049782; collision sphere radius=0.05326
- link mobilebase0_top_link: geometry collision sphere radius=0.078189; collision sphere radius=0.087608
Joints:
- removed joint gripperleft_0_eef_joint
- removed joint gripperright_0_eef_joint
- added joint gripper0_left_eef_joint: type fixed, parent robot0_left_hand, child gripper0_left_eef, origin xyz=0 0 0.097 rpy=0 0 -1.57079633
- added joint gripper0_right_eef_joint: type fixed, parent robot0_right_hand, child gripper0_right_eef, origin xyz=0 0 0.097 rpy=0 0 -1.57079633
